File: electronics/rgb-led-host/rgb-led-board/rgb-led-board.sch (KiCad schematic (older format))
At the start: 13 parts, among them P1 PAD_SOLDER_5mm, P2 PAD_SOLDER_5mm, P3 CONN_01X06, P4 PAD_SOLDER_5mm, P5 PAD_SOLDER_5mm, P6 PAD_SOLDER_5mm, P7 PAD_SOLDER_5mm, U1 AL1793AFE-13

Commit message: Updates to schematic and PCB layout
Routed and cosmetics placed.
Ready for fab exports.
Parts:
- removed C1: 100n_X7R_1005M, Applidyne_Capacitor:CAPC1005X60N, symbol appli_capacitor:100n_X7R_1005M
- removed P1, P2, P4, P5, P6, P7: PAD_SOLDER_5mm, Applidyne_Connector:PAD_SOLDER_5mm, symbol appli_connector:PAD_SOLDER_5mm
- removed P3: CONN_01X06, Applidyne_Connector_Wurth:61300611121, symbol appli_connector_wurth:CONN_01X06
- removed SL1: SOLDER-LINK-3, Applidyne_Link:SJ1608-3N, symbol appli_link:SOLDER-LINK-3
- added P1, P2, P4, P5, P6, P7: PAD_SOLDER_2mm, Applidyne_Connector:PAD_SOLDER_2mm, symbol appli_connector:PAD_SOLDER_2mm
- added P3: CONN_01X08, Applidyne_Connector_Wurth:61300811121, symbol appli_connector_wurth:CONN_01X08
- added SL1: SOLDER-LINK-2, Applidyne_Link:SJ1608-2N, symbol appli_link:SOLDER-LINK-2
- renumbered C2 to C1
Connections:
- net labels added: ~FAULT
- net labels removed: FAULT
- wire segments 43 -> 46
Other:
- note added: "Bridge for full output current."
- note added: "High to enable, internal PD"
- note added: "Open Drain, ASSERT LOW"
- note removed: "High to enable"
- note removed: "One jumper should be linked by default.\nBridge both for full output current."
- note removed: "Open Drain"
