File: electronics/esp32c6-internal-module/esp32c6-internal-module.kicad_sch (KiCad schematic)
At the start: 30 parts, among them J1 USB_C_SOCKET_RA_PTH_SIMPLE, P1 JST_SH_4_RA, P2 CONN_01X06, SW1 B3U-1000P_SPST-NO_SMD, SW2 B3U-1000P_SPST-NO_SMD, U1 ESP32-C6-MINI-1, U2 TLV76733DRV, U3 USBLC6

Commit message: Add manufacturing exports for C6 internal module board
Other:
- company: (none) -> S. RAPSON
- title: (none) -> ESP32-C6 DeltaBot Internal Module
Changed lines of the file:
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@@
 	(generator_version "8.0")
 	(paper "A4")
+	(title_block
+		(title "ESP32-C6 DeltaBot Internal Module")
+		(date "2024-06-18")
+		(rev "1.0")
+		(company "S. RAPSON")
+		(comment 3 "to provide WiFi or 802.15.4 bridged comms")
+		(comment 4 "Intended to connect to DeltaBot internal UART header")
+	)
 	(junction
 		(at 59.69 110.49)
